File: kicad/WS2812breakout/WS2812breakout.kicad_sch (KiCad schematic)
At the start: 3 parts, among them J3 Conn_01x04_Socket

Commit message: updated breakout schematic to include in/out lines
Connections:
- net I2C1_SCL is gone; now on net OUT: J3.3 (Pin_3)
- net OUT: now reaches D3.1 (DOUT)
- net I2C1_SDA renamed IN
- no-connect marks 2 -> 0
Changed lines of the file:
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@@
 		(color 0 0 0 0)
-	)
-	(no_connect
-		(at 219.71 127)
-	)
-	(no_connect
-		(at 203.2 100.33)
-	)
-	(wire
-		(pts
-			(xy 203.2 100.33) (xy 212.09 100.33)
-		)
-		(stroke
-			(width 0)
-			(type default)
-		)
 	)
 	(wire
@@
 		(pts
 			(xy 224.79 110.49) (xy 224.79 118.11)
+		)
+		(stroke
+			(width 0)
+			(type default)
+		)
+	)
+	(wire
+		(pts
+			(xy 203.2 100.33) (xy 212.09 100.33)
 		)
 		(stroke
@@
 	(wire
 		(pts
+			(xy 219.71 127) (xy 228.6 127)
+		)
+		(stroke
+			(width 0)
+			(type default)
+		)
+	)
+	(wire
+		(pts
 			(xy 203.2 97.79) (xy 212.09 97.79)
 		)
@@
 		)
 	)
-	(label "I2C1_SDA"
+	(label "OUT"
+		(at 203.2 100.33 0)
+		(fields_autoplaced yes)
+		(effects
+			(font
+				(size 1.27 1.27)
+			)
+			(justify left bottom)
+		)
+	)
+	(label "IN"
 		(at 203.2 97.79 0)
 		(fields_autoplaced yes)
@@
 		)
 	)
-	(label "I2C1_SCL"
-		(at 203.2 100.33 0)
+	(label "IN"
+		(at 191.77 127 0)
 		(fields_autoplaced yes)
 		(effects
@@
 		)
 	)
-	(label "I2C1_SDA"
-		(at 191.77 127 0)
+	(label "OUT"
+		(at 228.6 127 0)
 		(fields_autoplaced yes)
 		(effects

Commit message: final fixes
Parts:
- renumbered C7 to C1, D3 to D1, J3 to J1
Changed lines of the file:
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@@
 		(dnp no)
 		(fields_autoplaced yes)
-		(property "Reference" "#PWR021"
+		(property "Reference" "#PWR05"
 			(at 231.14 118.11 0)
 			(effects
@@
 			(project "WS2812breakout"
 				(path "/c3bd2aeb-acec-4e93-ab92-7a030f22ab8b"
-					(reference "#PWR021")
+					(reference "#PWR05")
 					(unit 1)
 				)
@@
 		(dnp no)
 		(fields_autoplaced yes)
-		(property "Reference" "#PWR027"
+		(property "Reference" "#PWR01"
 			(at 209.55 92.71 0)
 			(effects
@@
 			(project "WS2812breakout"
 				(path "/c3bd2aeb-acec-4e93-ab92-7a030f22ab8b"
-					(reference "#PWR027")
+					(reference "#PWR01")
 					(unit 1)
 				)
@@
 		(dnp no)
 		(fields_autoplaced yes)
-		(property "Reference" "#PWR020"
+		(property "Reference" "#PWR04"
 			(at 212.09 140.97 0)
 			(effects
@@
 			(project "WS2812breakout"
 				(path "/c3bd2aeb-acec-4e93-ab92-7a030f22ab8b"
-					(reference "#PWR020")
+					(reference "#PWR04")
 					(unit 1)
 				)
@@
 		(dnp no)
 		(fields_autoplaced yes)
-		(property "Reference" "J3"
+		(property "Reference" "J1"
 			(at 218.44 97.7899 0)
 			(effects
@@
 			(project "WS2812breakout"
 				(path "/c3bd2aeb-acec-4e93-ab92-7a030f22ab8b"
-					(reference "J3")
+					(reference "J1")
 					(unit 1)
 				)
@@
 		(on_board yes)
 		(dnp no)
-		(property "Reference" "D3"
+		(property "Reference" "D1"
 			(at 224.282 133.858 0)
 			(effects
@@
 			(project "WS2812breakout"
 				(path "/c3bd2aeb-acec-4e93-ab92-7a030f22ab8b"
-					(reference "D3")
+					(reference "D1")
 					(unit 1)
 				)
@@
 		(dnp no)
 		(fields_autoplaced yes)
-		(property "Reference" "#PWR019"
+		(property "Reference" "#PWR03"
 			(at 212.09 119.38 0)
 			(effects
@@
 			(project "WS2812breakout"
 				(path "/c3bd2aeb-acec-4e93-ab92-7a030f22ab8b"
-					(reference "#PWR019")
+					(reference "#PWR03")
 					(unit 1)
 				)
@@
 		(on_board yes)
 		(dnp no)
-		(property "Reference" "C7"
+		(property "Reference" "C1"
 			(at 220.218 116.586 90)
 			(effects
@@
 			(project "WS2812breakout"
 				(path "/c3bd2aeb-acec-4e93-ab92-7a030f22ab8b"
-					(reference "C7")
+					(reference "C1")
 					(unit 1)
 				)
@@
 		(dnp no)
 		(fields_autoplaced yes)
-		(property "Reference" "#PWR028"
+		(property "Reference" "#PWR02"
 			(at 199.39 102.87 0)
 			(effects
@@
 			(project "WS2812breakout"
 				(path "/c3bd2aeb-acec-4e93-ab92-7a030f22ab8b"
-					(reference "#PWR028")
-					(unit 1)
-				)
+					(reference "#PWR02")
+					(unit 1)
+				)
